Commit message: corrected lidar stl file name which is creating resolviing error in isaacsim

File: training/dynamic_obstacle_avoidance/source/dynamic_obstacle_avoidance/dynamic_obstacle_avoidance/assets/urdf/m3.urdf (robot description, URDF)
Before this commit: robot ROSMASTER-M3, 12 links, 11 joints
Links:
- link laser0_frame: geometry collision mesh filename=../meshes/Tmini_Plus2_1_Link.STL; visual mesh filename=../meshes/Tmini_Plus2_1_Link.STL
- link laser1_frame: geometry collision mesh filename=../meshes/Tmini_Plus2_2_Link.STL; visual mesh filename=../meshes/Tmini_Plus2_2_Link.STL
Joints:
- joint simcamera-Joint: axis 0 0 1 -> (none); type continuous -> fixed
