Commit message: added custom plugin to control the mecanum wheels

File: m3_ros2_ws/src/m3_ros2/urdf/ROSMASTER-M3.xacro (robot description, xacro)
@@ -9,3 +9,143 @@
   <xacro:common_base prefix="$(arg prefix)"  camera_type="$(arg camera_type)" /><!-- instantiated robot chassis -->
   <xacro:laser laser_type="$(arg laser_type)" prefix="$(arg prefix)" />         <!-- instantiate lidar -->
+  <!-- <ros2_control name="GazeboSystem" type="system">
+        <hardware>
+            <plugin>gz_ros2_control/GazeboSimSystem</plugin>
+        </hardware>
+    <joint name="$(arg prefix)lwheel1_Joint">
+      <command_interface name="velocity"/>
+      <state_interface name="velocity"/>
+      <state_interface name="position"/>
+    </joint>
+    <joint name="$(arg prefix)lwheel2_Joint">
+      <command_interface name="velocity"/>
+      <state_interface name="velocity"/>
+      <state_interface name="position"/>
+    </joint>
+    <joint name="$(arg prefix)rwheel1_Joint">
+      <command_interface name="velocity"/>
+      <state_interface name="velocity"/>
+      <state_interface name="position"/>
+    </joint>
+    <joint name="$(arg prefix)rwheel2_Joint">
+      <command_interface name="velocity"/>
+      <state_interface name="velocity"/>
+      <state_interface name="position"/>
+    </joint>
+  </ros2_control>
+  <gazebo>
+    <plugin
+        filename="gz_ros2_control-system"
+        name="gz_ros2_control::GazeboSimROS2ControlPlugin">
+        <parameters>$(find m3_ros2)/config/mecanum_controllers.yaml</parameters>
+    </plugin>
+  </gazebo> -->
+   <gazebo reference="$(arg prefix)lwheel1_Link">
+    <gravity>false</gravity>
+    <self_collide>false</self_collide>
+    <collision>
+      <surface>
+        <friction>
+          <ode>
+            <mu>0.0</mu>
+            <mu2>0.0</mu2>
+          </ode>
+        </friction>
+      </surface>
+    </collision>
+  </gazebo>
+     <gazebo reference="$(arg prefix)lwheel2_Link">
+    <gravity>false</gravity>
+    <self_collide>false</self_collide>
+    <collision>
+      <surface>
+        <friction>
+          <ode>
+            <mu>0.0</mu>
+            <mu2>0.0</mu2>
+          </ode>
+        </friction>
+      </surface>
+    </collision>
+  </gazebo>
+     <gazebo reference="$(arg prefix)rwheel1_Link">
+    <gravity>false</gravity>
+    <self_collide>false</self_collide>
+    <collision>
+      <surface>
+        <friction>
+          <ode>
+            <mu>0.0</mu>
+            <mu2>0.0</mu2>
+          </ode>
+        </friction>
+      </surface>
+    </collision>
+  </gazebo>
+     <gazebo reference="$(arg prefix)rwheel2_Link">
+    <gravity>false</gravity>
+    <self_collide>false</self_collide>
+    <collision>
+      <surface>
+        <friction>
+          <ode>
+            <mu>0.0</mu>
+            <mu2>0.0</mu2>
+          </ode>
+        </friction>
+      </surface>
+    </collision>
+  </gazebo>
+  <!-- <gazebo>
+  <plugin
+    filename="libkinematic_mecanum_system.so"
+    name="m3_kinematic_mecanum::KinematicMecanumSystem">
+    <topic>/cmd_vel</topic>
+    <base_link>$(arg prefix)base_link</base_link>
+    <front_left_joint>$(arg prefix)lwheel1_Joint</front_left_joint>
+    <rear_left_joint>$(arg prefix)lwheel2_Joint</rear_left_joint>
+    <front_right_joint>$(arg prefix)rwheel1_Joint</front_right_joint>
+    <rear_right_joint>$(arg prefix)rwheel2_Joint</rear_right_joint>
+    <wheel_radius>0.05</wheel_radius>
+    <wheel_base_x>0.0795</wheel_base_x>
+    <wheel_base_y>0.09775</wheel_base_y>
+  </plugin>
+</gazebo> -->
+<!-- Pose-based mecanum drive plugin (no ros2_control needed) -->
+  <gazebo>
+    <plugin
+      filename="libmecanum_pose_drive_system.so"
+      name="m3_mecanum_pose_drive::MecanumPoseDriveSystem">
+      <topic>/cmd_vel</topic>
+      <base_link>$(arg prefix)base_link</base_link>
+      <front_left_joint>$(arg prefix)lwheel1_Joint</front_left_joint>
+      <rear_left_joint>$(arg prefix)lwheel2_Joint</rear_left_joint>
+      <front_right_joint>$(arg prefix)rwheel1_Joint</front_right_joint>
+      <rear_right_joint>$(arg prefix)rwheel2_Joint</rear_right_joint>
+      <wheel_radius>0.05</wheel_radius>
+      <wheel_base_x>0.0795</wheel_base_x>
+      <wheel_base_y>0.09775</wheel_base_y>
+      <cmd_timeout>0.5</cmd_timeout>
+      <yaw_correction_gain>50.0</yaw_correction_gain>
+    </plugin>
+  </gazebo>
+  <!-- <gazebo>
+    <plugin
+      filename="gz-sim-mecanum-drive-system"
+      name="gz::sim::systems::MecanumDrive">
+      <front_left_joint>lwheel1_Joint</front_left_joint>
+      <back_left_joint>lwheel2_Joint</back_left_joint>
+      <front_right_joint>rwheel1_Joint</front_right_joint>
+      <back_right_joint>rwheel2_Joint</back_right_joint>
+      <wheel_separation>0.1955</wheel_separation>
+      <wheelbase>0.159</wheelbase>
+      <wheel_radius>0.05</wheel_radius>
+      <odom_publish_frequency>50</odom_publish_frequency>
+      <topic>cmd_vel</topic>
+      <odom_topic>odom</odom_topic>
+      <tf_topic>tf</tf_topic>
+      <frame_id>odom</frame_id>
+      <child_frame_id>base_link</child_frame_id>
+    </plugin>
+  </gazebo> -->
 </robot>

File: m3_ros2_ws/src/m3_ros2/urdf/common_base.xacro (robot description, xacro)
@@ -358,5 +358,5 @@
       link="${prefix}rwheel1_Link" />
     <axis
-      xyz="0 0 1" />
+      xyz="0 0 -1" />
   </joint>
   <!-- right rear wheel -->
@@ -412,5 +412,5 @@
       link="${prefix}rwheel2_Link" />
     <axis
-      xyz="0 0 1" />
+      xyz="0 0 -1" />
   </joint>
   </xacro:macro>
