Commit message: modified camera joint as fixed joint

File: m3_ros2_ws/src/m3_ros2/urdf/common_base.xacro (robot description, xacro)
@@ -118,5 +118,5 @@
     <joint
       name="${prefix}simcamera-Joint"
-      type="continuous">
+      type="fixed">
       <origin
         xyz="0 0 0"
@@ -126,6 +126,6 @@
       <child
         link="${prefix}ascamera_hp60c_camera_link_0" />
-      <axis
-        xyz="0 0 1" />
+      <!-- <axis
+        xyz="0 0 1" /> -->
     </joint>
   </xacro:if>
